Commit message: tf messages between the base link and the dvl link broadcasted

File: bluerov_model/BlueRov2.urdf.xacro (robot description, xacro)
@@ -82,5 +82,5 @@
     <origin xyz="0 0 0" rpy="0 3.141592653589793 -1.5707963267948966"/>
       <geometry>
-        <mesh filename="package://bluerov_ros_playground/model/BlueRov2.dae"/>
+        <mesh filename="package://waterlinked_a50_ros_driver/bluerov_model/BlueRov2.dae"/>
       </geometry>
     </visual>
